Commit message: finish navigation

File: src/jackal_description/urdf/accessories.urdf.xacro (robot description, xacro)
@@ -52,5 +52,5 @@
     <xacro:property name="prefix" value="$(optenv JACKAL_LASER_PREFIX ${mount})" />
     <xacro:property name="parent" value="$(optenv JACKAL_LASER_PARENT ${mount}_mount)" />
-    <xacro:property name="lidar_model" value="$(optenv JACKAL_LASER_MODEL tim551)" />
+    <xacro:property name="lidar_model" value="$(optenv JACKAL_LASER_MODEL utm30)" />
     <xacro:property name="mount_type" value="$(optenv JACKAL_LASER_MOUNT_TYPE upright)" />
     <!-- SICK LMS1xx -->
@@ -102,7 +102,102 @@
     </xacro:if>
     <!-- Hokuyo UTM30 -->
+    <!--
+    xacro:if value="${lidar_model == 'utm30'}">
+      <xacro:hokuyo_utm30_mount topic="${topic}" prefix="${prefix}" parent_link="${parent}">
+        <origin xyz="0 0 0.1" rpy="$(optenv JACKAL_LASER_RPY 0 0 0)" />
+      </xacro:hokuyo_utm30_mount>
+    </xacro:if>
+    -->
+    <!--new added for higher the UTM30 with the tower-->
+    <!-- Hokuyo UTM30 with custom tower (VLP16-style) -->
     <xacro:if value="${lidar_model == 'utm30'}">
-      <xacro:hokuyo_utm30_mount topic="${topic}" prefix="${prefix}" parent_link="${parent}">
-        <origin xyz="$(optenv JACKAL_LASER_OFFSET 0 0 0)" rpy="$(optenv JACKAL_LASER_RPY 0 0 0)" />
+      <xacro:property name="laser_height" value="0.1" />
+      <link name="${prefix}_utm30_mount"/>
+      <link name="${prefix}_utm30_plate">
+        <visual>
+          <geometry>
+            <box size="0.1 0.1 0.003"/>
+          </geometry>
+          <material name="black">
+            <color rgba="0 0 0 1" />
+          </material>
+        </visual>
+      </link>
+      <link name="${prefix}_utm30_leg1">
+        <visual>
+          <geometry>
+            <cylinder length="${laser_height}" radius="0.004"/>
+          </geometry>
+          <material name="white">
+            <color rgba="1 1 1 1" />
+          </material>
+          <origin xyz="0 0 ${laser_height/2}"/>
+        </visual>
+      </link>
+      <link name="${prefix}_utm30_leg2">
+        <visual>
+          <geometry>
+            <cylinder length="${laser_height}" radius="0.004"/>
+          </geometry>
+          <material name="white">
+            <color rgba="1 1 1 1" />
+          </material>
+          <origin xyz="0 0 ${laser_height/2}"/>
+        </visual>
+      </link>
+      <link name="${prefix}_utm30_leg3">
+        <visual>
+          <geometry>
+            <cylinder length="${laser_height}" radius="0.004"/>
+          </geometry>
+          <material name="white">
+            <color rgba="1 1 1 1" />
+          </material>
+          <origin xyz="0 0 ${laser_height/2}"/>
+        </visual>
+      </link>
+      <link name="${prefix}_utm30_leg4">
+        <visual>
+          <geometry>
+            <cylinder length="${laser_height}" radius="0.004"/>
+          </geometry>
+          <material name="white">
+            <color rgba="1 1 1 1" />
+          </material>
+          <origin xyz="0 0 ${laser_height/2}"/>
+        </visual>
+      </link>
+      <joint name="${prefix}_utm30_mount_joint" type="fixed">
+        <parent link="${parent}"/>
+        <child link="${prefix}_utm30_mount"/>
+        <origin xyz="0 0 0" rpy="0 0 0"/>
+      </joint>
+      <joint name="${prefix}_utm30_leg1_joint" type="fixed">
+        <parent link="${prefix}_utm30_mount"/>
+        <child link="${prefix}_utm30_leg1"/>
+        <origin xyz="0.05 0.05 0"/>
+      </joint>
+      <joint name="${prefix}_utm30_leg2_joint" type="fixed">
+        <parent link="${prefix}_utm30_mount"/>
+        <child link="${prefix}_utm30_leg2"/>
+        <origin xyz="0.05 -0.05 0"/>
+      </joint>
+      <joint name="${prefix}_utm30_leg3_joint" type="fixed">
+        <parent link="${prefix}_utm30_mount"/>
+        <child link="${prefix}_utm30_leg3"/>
+        <origin xyz="-0.05 0.05 0"/>
+      </joint>
+      <joint name="${prefix}_utm30_leg4_joint" type="fixed">
+        <parent link="${prefix}_utm30_mount"/>
+        <child link="${prefix}_utm30_leg4"/>
+        <origin xyz="-0.05 -0.05 0"/>
+      </joint>
+      <joint name="${prefix}_utm30_plate_joint" type="fixed">
+        <parent link="${prefix}_utm30_mount"/>
+        <child link="${prefix}_utm30_plate"/>
+        <origin xyz="0 0 ${laser_height}" rpy="0 0 0"/>
+      </joint>
+      <xacro:hokuyo_utm30_mount topic="${topic}" prefix="${prefix}" parent_link="${prefix}_utm30_plate">
+        <origin xyz="0 0 0" rpy="$(optenv JACKAL_LASER_RPY 0 0 0)" />
       </xacro:hokuyo_utm30_mount>
     </xacro:if>
@@ -260,4 +355,5 @@
   <xacro:include filename="$(find pointgrey_camera_description)/urdf/pointgrey_flea3.urdf.xacro" />
   <!-- If enabled, generate the flea3 camera payload with a tilt of 30 degrees. -->
+  <!--changed to invisible the white box-->
   <xacro:if value="$(optenv JACKAL_FLEA3 1)">
     <xacro:property name="name" value="$(optenv JACKAL_FLEA3_NAME front)" />

File: src/jackal_description/urdf/accessories/vlp16_mount.urdf.xacro (robot description, xacro)
@@ -10,5 +10,5 @@
           </geometry>
           <material name="black" />
-          <origin xyz="0 0 -0.001" rpy="0 0 0" />
+          <origin xyz="0 0 0" rpy="0 0 0" />
         </visual>
       </link>
@@ -16,10 +16,11 @@
         <visual>
           <geometry>
-            <cylinder length="${height}" radius="0.003" />
+            <!--changed the length of the leg-->
+            <cylinder length="${2*height}" radius="0.003" />
           </geometry>
           <material name="white">
             <color rgba="1 1 1 1" />
           </material>
-          <origin xyz="0 0 ${height/2}" rpy="0 0 0" />
+          <origin xyz="0 0 ${height}" rpy="0 0 0" />
         </visual>
       </link>
@@ -27,10 +28,10 @@
         <visual>
           <geometry>
-            <cylinder length="${height}" radius="0.003" />
+            <cylinder length="${2*height}" radius="0.003" />
           </geometry>
           <material name="white">
             <color rgba="1 1 1 1" />
           </material>
-          <origin xyz="0 0 ${height/2}" rpy="0 0 0" />
+          <origin xyz="0 0 ${height}" rpy="0 0 0" />
         </visual>
       </link>
@@ -38,10 +39,10 @@
         <visual>
           <geometry>
-            <cylinder length="${height}" radius="0.003" />
+            <cylinder length="${2*height}" radius="0.003" />
           </geometry>
           <material name="white">
             <color rgba="1 1 1 1" />
           </material>
-          <origin xyz="0 0 ${height/2}" rpy="0 0 0" />
+          <origin xyz="0 0 ${height}" rpy="0 0 0" />
         </visual>
       </link>
@@ -49,10 +50,10 @@
         <visual>
           <geometry>
-            <cylinder length="${height}" radius="0.003" />
+            <cylinder length="${2*height}" radius="0.003" />
           </geometry>
           <material name="white">
             <color rgba="1 1 1 1" />
           </material>
-          <origin xyz="0 0 ${height/2}" rpy="0 0 0" />
+          <origin xyz="0 0 ${height}" rpy="0 0 0" />
         </visual>
       </link>
@@ -85,5 +86,5 @@
         <parent link="${prefix}_vlp16_mount" />
         <child link="${prefix}_vlp16_plate" />
-        <origin xyz="0 0 ${height}" rpy="0 0 0" />
+        <origin xyz="0 0 ${2*height}" rpy="0 0 0" />
       </joint>
       <xacro:VLP-16 parent="${prefix}_vlp16_plate" topic="${topic}">

File: src/jackal_description/urdf/jackal.urdf.xacro (robot description, xacro)
@@ -1,4 +1,6 @@
 <?xml version="1.0"?>
 <robot name="jackal" xmlns:xacro="http://www.ros.org/wiki/xacro">
+  <!-- Kinect macro -->
+  <xacro:include filename="$(find jackal_description)/urdf/accessories/kinect_gazebo.xacro"/>
   <xacro:property name="PI" value="3.1415926535897931" />
   <xacro:property name="wheelbase" value="0.262" />
@@ -109,5 +111,5 @@
         iyy="0.3922" iyz="-0.0009"
         izz="0.4485"/>
-      </inertial>
+    </inertial>
   </link>
   <xacro:unless value="$(optenv JACKAL_FRONT_ACCESSORY_FENDER 0)">
@@ -218,9 +220,17 @@
     <origin xyz="${mount_spacing} 0 0" />
   </joint>
+  <!-- Kinect fixed on front_mount -->
+  <xacro:property name="kinect_offset_x" value="0.15"/>
+  <xacro:property name="kinect_offset_y" value="0.0"/>
+  <xacro:property name="kinect_offset_z" value="0.013"/>
+  <joint name="kinect_joint" type="fixed">
+    <origin xyz="${kinect_offset_x} ${kinect_offset_y} ${kinect_offset_z}" rpy="0 0 0"/>
+    <parent link="front_mount"/>
+    <child link="kinect_link"/>
+  </joint>
+  <xacro:kinect_camera prefix="kinect"/>
   <!-- Bring in simulation data for Gazebo. -->
   <xacro:include filename="$(find jackal_description)/urdf/jackal.gazebo" />
-  <!-- Optional standard accessories, including their simulation data. The rendering
-       of these into the final description is controlled by optenv variables, which
-       default each one to off.-->
+  <!-- Optional standard accessories, including their simulation data. -->
   <xacro:include filename="$(find jackal_description)/urdf/accessories.urdf.xacro" />
   <!-- Optional custom includes. -->
